Commit message: :FIX: Modify wrong tf frame

File: festival_r2/festival_ur_description/urdf/ur3e.urdf (robot description, URDF)
Before this commit: robot ur3e, 22 links, 21 joints
Links:
- removed link camera_bottom_screw_frame
- link camera_link: geometry collision box size=0.02505 0.025 0.09; visual mesh filename=package://festival_ur_description/meshes/sensors/d435.STL
- link display: geometry collision box size=0.2665 0.179 0.0615; visual mesh filename=package://festival_ur_description/meshes/ur3e/visual/displa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 scale=0.001 0.001 0.001
Joints:
- removed joint camera_joint
- joint camera_link_joint: origin xyz=0.010600000000000002 0.0175 0.0125 rpy=0 0 0 -> xyz=0.0135 0.0 -0.105 rpy=3.14159265359 0 0; parent camera_bottom_screw_frame -> display
- joint display_joint: origin xyz=0.0 0 0.0 rpy=0 0 0 -> xyz=0.0565 0 0.0 rpy=0 0 0
